File: rpi4b/shield_2024/shield_raspi.kicad_pcb (KiCad board)
At the start: 2 copper layers, 66 x 57 mm, 26 parts, among them J4 Conn_02x20_Odd_Even, U1 IRLML2402

Commit message: release V1
Parts:
- moved CLIM1 2.79 mm to (212.3, 85.3), turned to 0 degrees
Connections:
- CLIM1 pad 1: GND -> Net-(CLIM1-Pin_1)
- CLIM1 pad 2: Net-(CLIM1-Pin_2) -> +5V
- U1 pad 2: Net-(CLIM1-Pin_2) -> GND
- U1 pad 3: +5V -> Net-(CLIM1-Pin_1)
Routing:
- net Net-(CLIM1-Pin_1): track 0.00 -> 20.8 mm, vias 0 -> 1
- net Net-(CLIM1-Pin_2): track 19.4 -> 0.00 mm, vias 1 -> 0
- net +5V: track 98.7 -> 104.1 mm
Other:
- board text added: "UART GND|+5|+3.3|TX|RX"
- board text removed: "UART RX|TX|+3.3|+5|GND"
